File: controller/controller.kicad_sch (KiCad schematic)
At the start: 73 parts, among them J1 USB_A, J10 Conn_02x01, J11 Conn_02x01, J12 Conn_01x02, J13 Conn_01x01, J2 Conn_01x16, J3 Conn_01x16, J4 3.3V IO EXPANSION HEADER, J5 Conn_01x03, J6 DNP Conn_01x04, J7 Conn_02x01, J8 Conn_02x01, J9 Conn_02x01, SW1 SW_Push, U1 RP2040, U2 W25Q16JV, U3 74HC165, U4 USBLC6-2SC6, U5 DNP TXS0102DCU, U6 XC6206P332MR, Y1 12MHz

Commit message: Added LCSC part numbers for through-hole components
Parts:
- J1: LCSC (none) -> C3197751
- J2, J3: LCSC (none) -> C7191217
- J4: LCSC (none) -> C706867
